Commit message: new urdf

File: urdf/urdf/leg_left.xacro (robot description, xacro)
@@ -81,4 +81,12 @@
       </collision>
     </link>
+    <link name="${prefix}_FOOT_FINGER_00">
+      <collision>
+        <origin xyz="0 0 0" rpy="0 0 0"/>
+        <geometry>
+          <sphere radius="0.02"/>
+        </geometry>
+      </collision>
+    </link>
     <joint name="${prefix}_KFE" type="revolute">
       <origin xyz="0 0.303 0" rpy="0 0 0"/>
@@ -88,5 +96,5 @@
       <limit lower="${-130 *pi/180}" upper="${130 *pi/180}" effort="4800." velocity="7.4874625"/>
     </joint>
-    <joint name="${prefix}_FOOT" type="fixed">
+<!--     <joint name="${prefix}_FOOT" type="fixed">
       <origin xyz="0 0.17 0" rpy="${-pi/2} 0 0"/>
       <parent link="${prefix}_KFE"/>
@@ -94,6 +102,5 @@
       <axis xyz="0 0 1"/>
       <limit lower="${-16*pi/180}" upper="${16*pi/180}" effort="0" velocity="0"/>
-    </joint>
-    <!--
+    </joint> -->
     <joint name="${prefix}_ankle_1" type="revolute">
       <origin xyz="0 0.17 0" rpy="${-pi/2} 0 0"/>
@@ -118,20 +125,24 @@
       <axis xyz="0 0 1"/>
     </joint>
-    -->
     <joint name="${prefix}_finger_01" type="fixed">
-      <origin xyz="0.0482127 0.0876079 0.0389317" rpy="${pi} 0 0"/>
+      <origin xyz="0.0482127 0.0876079 0.04" rpy="${pi} 0 0"/>
       <parent link="${prefix}_FOOT"/>
       <child link="${prefix}_FOOT_FINGER_01"/>
     </joint>
     <joint name="${prefix}_finger_02" type="fixed">
-      <origin xyz="0.0491521 -0.0884335 0.0389153" rpy="${pi} 0 0"/>
+      <origin xyz="0.0491521 -0.0884335 0.04" rpy="${pi} 0 0"/>
       <parent link="${prefix}_FOOT"/>
       <child link="${prefix}_FOOT_FINGER_02"/>
     </joint>
     <joint name="${prefix}_finger_03" type="fixed">
-      <origin xyz="-0.1037888 0 0.0401649" rpy="${pi} 0 0"/>
+      <origin xyz="-0.1037888 0 0.04" rpy="${pi} 0 0"/>
       <parent link="${prefix}_FOOT"/>
       <child link="${prefix}_FOOT_FINGER_03"/>
     </joint>
+    <joint name="${prefix}_finger_00" type="fixed">
+      <origin xyz="0.0 0.0 0.04" rpy="${pi} 0 0"/>
+      <parent link="${prefix}_FOOT"/>
+      <child link="${prefix}_FOOT_FINGER_00"/>
+    </joint>
   </xacro:macro>
 </robot>

File: urdf/urdf/leg_right.xacro (robot description, xacro)
@@ -80,4 +80,12 @@
       </collision>
     </link>
+    <link name="${prefix}_FOOT_FINGER_00">
+      <collision>
+        <origin xyz="0 0 0" rpy="0 0 0"/>
+        <geometry>
+          <sphere radius="0.02"/>
+        </geometry>
+      </collision>
+    </link>
     <joint name="${prefix}_KFE" type="revolute">
       <origin xyz="0 0.303 0" rpy="0 0 0"/>
@@ -87,5 +95,4 @@
       <limit lower="${-130 *pi/180}" upper="${130 *pi/180}" effort="4800." velocity="7.4874625"/>
     </joint>
-    <!--
     <joint name="${prefix}_ankle_1" type="revolute">
       <origin xyz="0 0.17 0" rpy="${-pi/2} 0 0"/>
@@ -110,6 +117,5 @@
       <axis xyz="0 0 1"/>
     </joint>
-    -->
-    <joint name="${prefix}_FOOT" type="fixed">
+<!--     <joint name="${prefix}_FOOT" type="fixed">
       <origin xyz="0 0.17 0" rpy="${-pi/2} 0 0"/>
       <parent link="${prefix}_KFE"/>
@@ -117,20 +123,25 @@
       <axis xyz="0 0 1"/>
       <limit lower="${-16*pi/180}" upper="${16*pi/180}" effort="0" velocity="0"/>
-    </joint>
+    </joint> -->
     <joint name="${prefix}_finger_01" type="fixed">
-      <origin xyz="0.0482127 0.0876079 0.0389317" rpy="${pi} 0 0"/>
+      <origin xyz="0.0482127 0.0876079 0.04" rpy="${pi} 0 0"/>
       <parent link="${prefix}_FOOT"/>
       <child link="${prefix}_FOOT_FINGER_01"/>
     </joint>
     <joint name="${prefix}_finger_02" type="fixed">
-      <origin xyz="0.0491521 -0.0884335 0.0389153" rpy="${pi} 0 0"/>
+      <origin xyz="0.0491521 -0.0884335 0.04" rpy="${pi} 0 0"/>
       <parent link="${prefix}_FOOT"/>
       <child link="${prefix}_FOOT_FINGER_02"/>
     </joint>
     <joint name="${prefix}_finger_03" type="fixed">
-      <origin xyz="-0.1037888 0 0.0401649" rpy="${pi} 0 0"/>
+      <origin xyz="-0.1037888 0 0.040" rpy="${pi} 0 0"/>
       <parent link="${prefix}_FOOT"/>
       <child link="${prefix}_FOOT_FINGER_03"/>
     </joint>
+    <joint name="${prefix}_finger_00" type="fixed">
+      <origin xyz="0.0 0.0 0.04" rpy="${pi} 0 0"/>
+      <parent link="${prefix}_FOOT"/>
+      <child link="${prefix}_FOOT_FINGER_00"/>
+    </joint>
   </xacro:macro>
 </robot>
